File: EAGLE/projects/Blueshift 2/pcb_1love.brd (EAGLE design)
At the start: 96.5 x 226.7 mm, 20 parts, among them X1 RASPI_BOARD_B+_F

Commit message: Fix issue where power and ground aren't connected the Fathom X
Connections:
- net +12V: now also U$1.VIN
- net GND: now also U$1.GND
Changed lines of the file:
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@@
 </layers>
 <board>
-<fusionsync huburn="a.YnVzaW5lc3M6Z21haWw4NTczMzE" projecturn="a.YnVzaW5lc3M6Z21haWw4NTczMzEjMjAyMDA1MDQyOTQ0NDQ1MDE" f3durn="urn:adsk.wipprod:dm.lineage:yFlxF8sUSF--vyBRsOsgSQ" pcbguid="" lastpulledtime="" lastsyncedchangeguid="" latestrevisionid="d2326aaf-4f00-4cae-a935-0311d6c788cf" lastsyncedrevisionid="d2326aaf-4f00-4cae-a935-0311d6c788cf" lastboardhashguid="c0c99a6b-c641-34e0-a0ba-0d49286527be" lastpushedtime="2020-05-08T17:41:11Z" linktopcb3d="%12"/>
 <plain>
 <wire x1="96.52" y1="0" x2="96.52" y2="164.465" width="0" layer="20"/>
@@
 </autorouter>
 <elements>
-<element name="BT_ESC_A" library="BlueShift" package="2CONTAC_ULTRAFIT_R/A" value="" x="12.7" y="130.81" smashed="yes" rot="MR0">
+<element name="BT_ESC_A" library="BlueShift" package="2CONTAC_ULTRAFIT_R/A" package3d_urn="urn:adsk.eagle:package:19990303/3" value="" x="12.7" y="130.81" smashed="yes" rot="MR0">
 <attribute name="NAME" x="16.51" y="130.81" size="1.27" layer="26" rot="MR0"/>
 <attribute name="VALUE" x="16.51" y="113.03" size="1.27" layer="26" rot="MR0"/>
 </element>
-<element name="BT_ESC_B" library="BlueShift" package="2CONTAC_ULTRAFIT_R/A" value="" x="24.13" y="113.03" smashed="yes" rot="MR0">
+<element name="BT_ESC_B" library="BlueShift" package="2CONTAC_ULTRAFIT_R/A" package3d_urn="urn:adsk.eagle:package:19990303/3" value="" x="24.13" y="113.03" smashed="yes" rot="MR0">
 <attribute name="NAME" x="27.94" y="113.03" size="1.27" layer="26" rot="MR0"/>
 <attribute name="VALUE" x="27.94" y="95.25" size="1.27" layer="26" rot="MR0"/>
 </element>
-<element name="BT_ESC_C" library="BlueShift" package="2CONTAC_ULTRAFIT_R/A" value="" x="41.91" y="130.81" smashed="yes" rot="MR0">
+<element name="BT_ESC_C" library="BlueShift" package="2CONTAC_ULTRAFIT_R/A" package3d_urn="urn:adsk.eagle:package:19990303/3" value="" x="41.91" y="130.81" smashed="yes" rot="MR0">
 <attribute name="NAME" x="45.72" y="130.81" size="1.27" layer="26" rot="MR0"/>
 <attribute name="VALUE" x="45.72" y="113.03" size="1.27" layer="26" rot="MR0"/>
 </element>
-<element name="BT_ESC_D" library="BlueShift" package="2CONTAC_ULTRAFIT_R/A" value="" x="57.15" y="113.03" smashed="yes" rot="MR0">
+<element name="BT_ESC_D" library="BlueShift" package="2CONTAC_ULTRAFIT_R/A" package3d_urn="urn:adsk.eagle:package:19990303/3" value="" x="57.15" y="113.03" smashed="yes" rot="MR0">
 <attribute name="NAME" x="60.96" y="113.03" size="1.27" layer="26" rot="MR0"/>
 <attribute name="VALUE" x="60.96" y="95.25" size="1.27" layer="26" rot="MR0"/>
 </element>
-<element name="BT_ESC_E" library="BlueShift" package="2CONTAC_ULTRAFIT_R/A" value="" x="76.2" y="130.81" smashed="yes" rot="MR0">
+<element name="BT_ESC_E" library="BlueShift" package="2CONTAC_ULTRAFIT_R/A" package3d_urn="urn:adsk.eagle:package:19990303/3" value="" x="76.2" y="130.81" smashed="yes" rot="MR0">
 <attribute name="NAME" x="80.01" y="130.81" size="1.27" layer="26" rot="MR0"/>
 <attribute name="VALUE" x="80.01" y="113.03" size="1.27" layer="26" rot="MR0"/>
 </element>
-<element name="BT_ESC_F" library="BlueShift" package="2CONTAC_ULTRAFIT_R/A" value="" x="90.17" y="113.03" smashed="yes" rot="MR0">
+<element name="BT_ESC_F" library="BlueShift" package="2CONTAC_ULTRAFIT_R/A" package3d_urn="urn:adsk.eagle:package:19990303/3" value="" x="90.17" y="113.03" smashed="yes" rot="MR0">
 <attribute name="NAME" x="93.98" y="113.03" size="1.27" layer="26" rot="MR0"/>
 <attribute name="VALUE" x="93.98" y="95.25" size="1.27" layer="26" rot="MR0"/>
 </element>
-<element name="CONN13" library="BlueShift" package="2CONTAC_ULTRAFIT_R/A" value="" x="7.62" y="16.51" smashed="yes">
+<element name="CONN13" library="BlueShift" package="2CONTAC_ULTRAFIT_R/A" package3d_urn="urn:adsk.eagle:package:19990303/3" value="" x="7.62" y="16.51" smashed="yes">
 <attribute name="NAME" x="3.81" y="16.51" size="1.27" layer="25"/>
 <attribute name="VALUE" x="3.81" y="-1.27" size="1.27" layer="25"/>
 </element>
-<element name="CONN14" library="BlueShift" package="2CONTAC_ULTRAFIT_R/A" value="" x="72.39" y="151.13" smashed="yes">
+<element name="CONN14" library="BlueShift" package="2CONTAC_ULTRAFIT_R/A" package3d_urn="urn:adsk.eagle:package:19990303/3" value="" x="72.39" y="151.13" smashed="yes">
 <attribute name="NAME" x="68.58" y="151.13" size="1.27" layer="25"/>
 <attribute name="VALUE" x="68.58" y="133.35" size="1.27" layer="25"/>
@@
 <attribute name="VALUE" x="57.785" y="193.675" size="1.27" layer="25" rot="R270"/>
 </element>
-<element name="POWER-IN" library="BlueShift" package="2-CONTACT-SUPER" value="" x="73.66" y="3.81" smashed="yes" rot="R180"/>
+<element name="POWER-IN" library="BlueShift" package="2-CONTACT-SUPER" package3d_urn="urn:adsk.eagle:package:19991152/2" value="" x="73.66" y="3.81" smashed="yes" rot="R180"/>
 <element name="PWM_EXT" library="BlueShift" package="PWM_EXTENDER-SIMPLE" value="" x="89.535" y="218.44" smashed="yes" rot="MR270">
 <attribute name="NAME" x="69.215" y="193.04" size="1.27" layer="22" rot="MR270"/>
 <attribute name="VALUE" x="98.425" y="193.04" size="1.27" layer="22" rot="MR270"/>
 </element>
-<element name="TP_ESC_A" library="BlueShift" package="2CONTAC_ULTRAFIT_R/A" value="" x="12.7" y="113.03" smashed="yes">
+<element name="TP_ESC_A" library="BlueShift" package="2CONTAC_ULTRAFIT_R/A" package3d_urn="urn:adsk.eagle:package:19990303/3" value="" x="12.7" y="113.03" smashed="yes">
 <attribute name="NAME" x="8.89" y="113.03" size="1.27" layer="25"/>
+<attribute name="SPICEPREFIX" value="B" x="12.7" y="113.03" size="1.778" layer="27" display="off"/>
 <attribute name="VALUE" x="8.89" y="95.25" size="1.27" layer="25"/>
 </element>
-<element name="TP_ESC_B" library="BlueShift" package="2CONTAC_ULTRAFIT_R/A" value="" x="24.13" y="130.81" smashed="yes">
+<element name="TP_ESC_B" library="BlueShift" package="2CONTAC_ULTRAFIT_R/A" package3d_urn="urn:adsk.eagle:package:19990303/3" value="" x="24.13" y="130.81" smashed="yes">
 <attribute name="NAME" x="20.32" y="130.81" size="1.27" layer="25"/>
 <attribute name="VALUE" x="20.32" y="113.03" size="1.27" layer="25"/>
 </element>
-<element name="TP_ESC_C" library="BlueShift" package="2CONTAC_ULTRAFIT_R/A" value="" x="41.91" y="113.03" smashed="yes">
+<element name="TP_ESC_C" library="BlueShift" package="2CONTAC_ULTRAFIT_R/A" package3d_urn="urn:adsk.eagle:package:19990303/3" value="" x="41.91" y="113.03" smashed="yes">
 <attribute name="NAME" x="38.1" y="113.03" size="1.27" layer="25"/>
 <attribute name="VALUE" x="38.1" y="95.25" size="1.27" layer="25"/>
 </element>
-<element name="TP_ESC_D" library="BlueShift" package="2CONTAC_ULTRAFIT_R/A" value="" x="57.15" y="130.81" smashed="yes">
+<element name="TP_ESC_D" library="BlueShift" package="2CONTAC_ULTRAFIT_R/A" package3d_urn="urn:adsk.eagle:package:19990303/3" value="" x="57.15" y="130.81" smashed="yes">
 <attribute name="NAME" x="53.34" y="130.81" size="1.27" layer="25"/>
 <attribute name="VALUE" x="53.34" y="113.03" size="1.27" layer="25"/>
 </element>
-<element name="TP_ESC_E" library="BlueShift" package="2CONTAC_ULTRAFIT_R/A" value="" x="76.2" y="113.03" smashed="yes">
+<element name="TP_ESC_E" library="BlueShift" package="2CONTAC_ULTRAFIT_R/A" package3d_urn="urn:adsk.eagle:package:19990303/3" value="" x="76.2" y="113.03" smashed="yes">
 <attribute name="NAME" x="72.39" y="113.03" size="1.27" layer="25"/>
 <attribute name="VALUE" x="72.39" y="95.25" size="1.27" layer="25"/>
 </element>
-<element name="TP_ESC_F" library="BlueShift" package="2CONTAC_ULTRAFIT_R/A" value="" x="90.17" y="130.81" smashed="yes">
+<element name="TP_ESC_F" library="BlueShift" package="2CONTAC_ULTRAFIT_R/A" package3d_urn="urn:adsk.eagle:package:19990303/3" value="" x="90.17" y="130.81" smashed="yes">
 <attribute name="NAME" x="86.36" y="130.81" size="1.27" layer="25"/>
 <attribute name="VALUE" x="86.36" y="113.03" size="1.27" layer="25"/>
@@
 <vertex x="-6.35" y="233.68"/>
 </polygon>
+<contactref element="U$1" pad="GND"/>
 </signal>
 <signal name="+12V">
@@
 <vertex x="-5.08" y="233.68"/>
 </polygon>
+<contactref element="U$1" pad="VIN"/>
 </signal>
 <signal name="+24V">
@@
 <compatibility>
 <note version="8.3" severity="warning">
-Since Version 8.3, EAGLE supports Fusion synchronisation.
-This feature will not be available in this version and saving
-the document will break the link to the Fusion PCB feature.
+Since Version 8.3, EAGLE supports URNs for individual library
+assets (packages, symbols, and devices). The URNs of those assets
+will not be understood (or retained) with this version.
+</note>
+<note version="8.3" severity="warning">
+Since Version 8.3, EAGLE supports the association of 3D packages
+with devices in libraries, schematics, and board files. Those 3D
+packages will not be understood (or retained) with this version.
 </note>
 </compatibility>
