File: EAGLE/projects/Blueshift 2/pcb_1love.sch (EAGLE design)
At the start: 20 parts, among them X1 RASPI_BOARD_B+_F

Commit message: Fix issue where power and ground aren't connected the Fathom X
Parts:
- TP_ESC_A: SPICEPREFIX (none) -> B
Connections:
- net +12V: now also U$1.VIN
- net GND: now also U$1.GND
Other:
- moved on the sheet: U$1
Changed lines of the file:
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@@
 <part name="U$1" library="FathomX" deviceset="FATHOM-X" device=""/>
 <part name="X1" library="raspberrypi" deviceset="RASPI_BOARD_B+" device="_F"/>
-<part name="POWER-IN" library="BlueShift" deviceset="2-CONTACT-SUPER" device=""/>
-<part name="TP_ESC_A" library="BlueShift" deviceset="2CONTACT_ULTRAFIT_R/A" device=""/>
-<part name="TP_ESC_B" library="BlueShift" deviceset="2CONTACT_ULTRAFIT_R/A" device=""/>
-<part name="TP_ESC_C" library="BlueShift" deviceset="2CONTACT_ULTRAFIT_R/A" device=""/>
-<part name="TP_ESC_D" library="BlueShift" deviceset="2CONTACT_ULTRAFIT_R/A" device=""/>
-<part name="TP_ESC_E" library="BlueShift" deviceset="2CONTACT_ULTRAFIT_R/A" device=""/>
-<part name="BT_ESC_A" library="BlueShift" deviceset="2CONTACT_ULTRAFIT_R/A" device=""/>
-<part name="BT_ESC_B" library="BlueShift" deviceset="2CONTACT_ULTRAFIT_R/A" device=""/>
-<part name="BT_ESC_C" library="BlueShift" deviceset="2CONTACT_ULTRAFIT_R/A" device=""/>
-<part name="BT_ESC_D" library="BlueShift" deviceset="2CONTACT_ULTRAFIT_R/A" device=""/>
-<part name="BT_ESC_E" library="BlueShift" deviceset="2CONTACT_ULTRAFIT_R/A" device=""/>
-<part name="BT_ESC_F" library="BlueShift" deviceset="2CONTACT_ULTRAFIT_R/A" device=""/>
-<part name="TP_ESC_F" library="BlueShift" deviceset="2CONTACT_ULTRAFIT_R/A" device=""/>
-<part name="CONN13" library="BlueShift" deviceset="2CONTACT_ULTRAFIT_R/A" device=""/>
+<part name="POWER-IN" library="BlueShift" deviceset="2-CONTACT-SUPER" device="" package3d_urn="urn:adsk.eagle:package:19991152/2"/>
+<part name="TP_ESC_A" library="BlueShift" deviceset="2CONTACT_ULTRAFIT_R/A" device="" package3d_urn="urn:adsk.eagle:package:19990303/3">
+<attribute name="SPICEPREFIX" value="B"/>
+</part>
+<part name="TP_ESC_B" library="BlueShift" deviceset="2CONTACT_ULTRAFIT_R/A" device="" package3d_urn="urn:adsk.eagle:package:19990303/3"/>
+<part name="TP_ESC_C" library="BlueShift" deviceset="2CONTACT_ULTRAFIT_R/A" device="" package3d_urn="urn:adsk.eagle:package:19990303/3"/>
+<part name="TP_ESC_D" library="BlueShift" deviceset="2CONTACT_ULTRAFIT_R/A" device="" package3d_urn="urn:adsk.eagle:package:19990303/3"/>
+<part name="TP_ESC_E" library="BlueShift" deviceset="2CONTACT_ULTRAFIT_R/A" device="" package3d_urn="urn:adsk.eagle:package:19990303/3"/>
+<part name="BT_ESC_A" library="BlueShift" deviceset="2CONTACT_ULTRAFIT_R/A" device="" package3d_urn="urn:adsk.eagle:package:19990303/3"/>
+<part name="BT_ESC_B" library="BlueShift" deviceset="2CONTACT_ULTRAFIT_R/A" device="" package3d_urn="urn:adsk.eagle:package:19990303/3"/>
+<part name="BT_ESC_C" library="BlueShift" deviceset="2CONTACT_ULTRAFIT_R/A" device="" package3d_urn="urn:adsk.eagle:package:19990303/3"/>
+<part name="BT_ESC_D" library="BlueShift" deviceset="2CONTACT_ULTRAFIT_R/A" device="" package3d_urn="urn:adsk.eagle:package:19990303/3"/>
+<part name="BT_ESC_E" library="BlueShift" deviceset="2CONTACT_ULTRAFIT_R/A" device="" package3d_urn="urn:adsk.eagle:package:19990303/3"/>
+<part name="BT_ESC_F" library="BlueShift" deviceset="2CONTACT_ULTRAFIT_R/A" device="" package3d_urn="urn:adsk.eagle:package:19990303/3"/>
+<part name="TP_ESC_F" library="BlueShift" deviceset="2CONTACT_ULTRAFIT_R/A" device="" package3d_urn="urn:adsk.eagle:package:19990303/3"/>
+<part name="CONN13" library="BlueShift" deviceset="2CONTACT_ULTRAFIT_R/A" device="" package3d_urn="urn:adsk.eagle:package:19990303/3"/>
 <part name="GND1" library="supply1" library_urn="urn:adsk.eagle:library:371" deviceset="GND" device=""/>
 <part name="GND2" library="supply1" library_urn="urn:adsk.eagle:library:371" deviceset="GND" device=""/>
@@
 <part name="GND17" library="supply1" library_urn="urn:adsk.eagle:library:371" deviceset="GND" device=""/>
 <part name="GND18" library="supply1" library_urn="urn:adsk.eagle:library:371" deviceset="GND" device=""/>
-<part name="CONN14" library="BlueShift" deviceset="2CONTACT_ULTRAFIT_R/A" device=""/>
+<part name="CONN14" library="BlueShift" deviceset="2CONTACT_ULTRAFIT_R/A" device="" package3d_urn="urn:adsk.eagle:package:19990303/3"/>
 <part name="GND19" library="supply1" library_urn="urn:adsk.eagle:library:371" deviceset="GND" device=""/>
 <part name="P+21" library="supply1" library_urn="urn:adsk.eagle:library:371" deviceset="+12V" device=""/>
@@
 <instance part="U$1" gate="G$1" x="33.02" y="91.44" smashed="yes" rot="R270">
 <attribute name="NAME" x="43.18" y="73.66" size="1.27" layer="95" rot="R270"/>
-<attribute name="VALUE" x="10.16" y="73.66" size="1.27" layer="96" rot="R270"/>
+<attribute name="VALUE" x="38.1" y="76.2" size="1.27" layer="96" rot="R270"/>
 </instance>
 <instance part="X1" gate="G$1" x="33.02" y="127" smashed="yes"/>
@@
 <pinref part="CONN14" gate="G$1" pin="1"/>
 </segment>
+<segment>
+<pinref part="U$1" gate="G$1" pin="GND"/>
+<pinref part="GND15" gate="1" pin="GND"/>
+</segment>
 </net>
 <net name="+12V" class="0">
@@
 <pinref part="VCONVERTER" gate="G$1" pin="VIN"/>
 </segment>
+<segment>
+<pinref part="U$1" gate="G$1" pin="VIN"/>
+<pinref part="P+22" gate="1" pin="+12V"/>
+</segment>
 </net>
 <net name="+24V" class="0">
@@
 <pinref part="CONN13" gate="G$1" pin="2"/>
 <pinref part="U$1" gate="G$1" pin="PL_L"/>
-<wire x1="2.54" y1="73.66" x2="33.02" y2="73.66" width="0.1524" layer="91"/>
+<wire x1="2.54" y1="73.66" x2="27.94" y2="73.66" width="0.1524" layer="91"/>
 </segment>
 </net>
@@
 <segment>
 <pinref part="U$1" gate="G$1" pin="HV_SIGNAL"/>
-<wire x1="33.02" y1="71.12" x2="7.62" y2="71.12" width="0.1524" layer="91"/>
+<wire x1="27.94" y1="71.12" x2="7.62" y2="71.12" width="0.1524" layer="91"/>
 <wire x1="7.62" y1="71.12" x2="7.62" y2="68.58" width="0.1524" layer="91"/>
 <pinref part="CONN13" gate="G$1" pin="1"/>
@@
 will not be understood (or retained) with this version.
 </note>
+<note version="8.3" severity="warning">
+Since Version 8.3, EAGLE supports the association of 3D packages
+with devices in libraries, schematics, and board files. Those 3D
+packages will not be understood (or retained) with this version.
+</note>
 </compatibility>
